File: KiCad_Archives/ElectricKettle.sch (KiCad schematic (older format))
At the start: 44 parts, among them IC1 ATMEGA328-P, J1 Termocouple_Shield_Header, P1 LOAD_OUT, P2 127VAC, P3 WATER_SENSOR_IN, P4 ON/OFF SW, Q1 TRIAC_BTA, SW1 RESET, SW2 TEMP+, SW3 TEMP-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

Commit message: ADD: All Fabrication Files
Parts:
- added C11: 100n, symbol C_Small
- added P5: FT232_MODULE, symbol CONN_01X06
- added R12: 100k, w_pth_resistors:RC03, symbol R
- R1, R10, R11, R2, R3, R4, R5, R7, R8, R9, Y1: footprint (none) -> w_pth_resistors:RC03
- R6: value R -> 20k; footprint (none) -> w_pth_resistors:RC03
- RV1: value POT -> 5k; footprint (none) -> w_pth_resistors:RC03
- U3: footprint (none) -> TO_SOT_Packages_THT:TO-220-3_Vertical
Connections:
- net SDO is gone; now on net MISO: J1.15 (SDO)
- net +5V: now also RV1.1, P5.4 (P4)
- net GND: now also RV1.3, P5.6 (P6), R12.2
- net POWER_IN1: now also F2.2, T1.1 (AA)
- net POWER_IN2: now also P4.1 (P1), T1.2 (AB), U1.4
- net RX: now also P5.3 (P3)
- net TX: now also P5.2 (P2)
- net WAVE_FEEDBACK: now also U2.5; no longer U2.6
- net ~RESET: now also C11.1
- new net CTS: P5.5 (P5), R12.1
- new net DTR: C11.2, P5.1 (P1)
- no-connect marks 29 -> 30
Other:
- note added: "FT232 Serial Connections"
- moved on the sheet: C10, C7, C8, C9, D2, D3, DS1, F1, F2, P2, P3, P4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
